File: pcb/F407-v10/CanShark.sch (EAGLE design)
At the start: 129 parts, among them IC1 STM32F407V, IC2 KSZ8051MLL, K2 JACK_POWER_2,1, U1 SN65HVD230DR, U2 SN65HVD230DR, U3 LM2594M-ADJ, U4 LM2594M-ADJ, U5 TSH24IDT, U6 MCP602-E/SN

Commit message: [pcb] change texts of PCB
Parts:
- C27, C28: value (none) -> 100uF/16V
- C29, C38: value (none) -> 100uF/20V
- C35, C9: value 10nF -> 100nF
- D1, D2: value (none) -> SK26A
- L3: value (none) -> 68uH
- L4: value (none) -> 100uH
- R59: value 200k -> 100k
Other:
- moved on the sheet: C11, C12, C13, C14, C15, C16, C17, C18, C19, C20, C21, C22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
